Commit message: Fixed kinect description

File: tutorial_commons/urdf/kinect.xacro (robot description, xacro)
@@ -41,5 +41,5 @@
      <origin xyz="0 0 0" rpy="0 0 ${M_PI/2}"/>
       <geometry>
-       <mesh filename="package://tutorial_commons/meshes/sensors/kinect.dae"/>
+       <mesh filename="package://tutorial_commons/meshes/kinect.dae"/>
       </geometry>
     </visual>
